Commit message: implemented PID controller with underside camera

File: agrobot_ws/src/agrobot/urdf/robot.xacro (robot description, xacro)
@@ -186,4 +186,18 @@
       <geometry>
         <box size="${camera_length} ${camera_width} ${camera_height}"/>
+      </geometry>
+    </visual>
+  </link>
+  <link name='downward_camera_link'>
+    <xacro:box_inertial name="downward_camera_link" m="${camera_mass}" x="${camera_width}" y="${camera_length}" z="${camera_height}"/>
+    <collision name='downward_camera_link_collision'>
+      <geometry>
+        <box size="${camera_length} ${camera_width} ${camera_height}"/>
+      </geometry>
+    </collision>
+    <visual name='camera_link_visual'>
+      <origin xyz="0 0 0" rpy=" 0 ${3.1415926/2} 0"/>
+      <geometry>
+        <box size="${5*camera_length} ${2*camera_width} ${camera_height}"/>
       </geometry>
     </visual>
@@ -265,4 +279,49 @@
   </sensor>
   </gazebo>
+  <joint name="downward_camera_joint" type="fixed">
+    <parent link="chassis"/>
+    <child link="downward_camera_link"/>
+    <origin xyz="0 0 ${-3*camera_height}" rpy="0 1.57 0"/>
+  </joint>
+  <gazebo reference="downward_camera_link">
+    <material>Gazebo/Red</material>
+    <sensor type="camera" name="downward_camera_link">
+    <update_rate>30.0</update_rate>
+    <camera name="head">
+      <horizontal_fov>1.3962634</horizontal_fov>
+      <image>
+        <width>800</width>
+        <height>800</height>
+        <format>R8G8B8</format>
+      </image>
+      <clip>
+        <near>0.02</near>
+        <far>300</far>
+      </clip>
+      <noise>
+        <type>gaussian</type>
+        <!-- Noise is sampled independently per pixel on each frame.
+              That pixel's noise value is added to each of its color
+              channels, which at that point lie in the range [0,1]. -->
+        <mean>0.0</mean>
+        <stddev>0.007</stddev>
+      </noise>
+    </camera>
+    <plugin name="camera_controller" filename="libgazebo_ros_camera.so">
+      <alwaysOn>true</alwaysOn>
+      <updateRate>0.0</updateRate>
+      <cameraName>robot/downward_camera</cameraName>
+      <imageTopicName>downward_image_raw</imageTopicName>
+      <cameraInfoTopicName>downward_camera_info</cameraInfoTopicName>
+      <frameName>downward_camera_link</frameName>
+      <hackBaseline>0.07</hackBaseline>
+      <distortionK1>0.0</distortionK1>
+      <distortionK2>0.0</distortionK2>
+      <distortionK3>0.0</distortionK3>
+      <distortionT1>0.0</distortionT1>
+      <distortionT2>0.0</distortionT2>
+    </plugin>
+  </sensor>
+  </gazebo>
   <gazebo reference="wheel_FL">
     <material>Gazebo/Yellow</material>

Commit message: most recent gazebo changes + started algorithm for downward image

File: agrobot_ws/src/agrobot/urdf/robot.xacro (robot description, xacro)
@@ -9,5 +9,6 @@
   <xacro:property name="chassis_height" value="0.05"/>
   <xacro:property name="chassis_mass" value="1.0"/>
-  <xacro:property name="wheel_radius" value="0.0425"/>
+  <xacro:property name="wheel_radius" value="0.1"/>
+  <!-- 0.0425 -->
   <xacro:property name="wheel_width" value="0.03"/>
   <xacro:property name="wheel_mass" value="0.5"/>
@@ -334,5 +335,5 @@
   </gazebo>
   <gazebo reference="wheel_RR">
-    <material>Gazebo/Yellow</material>
+    <material>Gazebo/Black</material>
   </gazebo>
   <gazebo>
@@ -344,10 +345,17 @@
       <leftRearJoint>wheel_RL_joint</leftRearJoint>
       <rightRearJoint>wheel_RR_joint</rightRearJoint>
-      <wheelSeparation>0.4</wheelSeparation>
+      <wheelSeparation>0.5</wheelSeparation>
+      <!-- 0.4 -->
       <wheelDiameter>0.215</wheelDiameter>
       <robotBaseFrame>base_link</robotBaseFrame>
-      <torque>20</torque>
+      <torque>1000</torque>
       <topicName>cmd_vel</topicName>
       <broadcastTF>false</broadcastTF>
+      <kp>1000000.0</kp> <!-- kp and kd for rubber -->
+      <kd>100.0</kd>
+      <mu1>1.0</mu1>
+      <mu2>1.0</mu2>
+      <maxVel>1.0</maxVel>
+      <minDepth>0.00</minDepth>
     </plugin>
   </gazebo>

File: agrobot_ws/src/agrobot/urdf/wheel.xacro (robot description, xacro)
@@ -34,321 +34,29 @@
       </material>
     </visual>
-  </link>
-  <link name='leg_FR'>
-    <xacro:box_inertial name="leg_FR" m="${leg_mass}" x="${leg_length}" y="${leg_width}" z="${leg_height}"/>
-    <collision name='leg_FR_collision'>
-      <origin xyz="0 0 0" rpy="0 0 0"/>
-      <geometry>
-        <box size="${leg_length} ${leg_width} ${leg_height}"/>
-      </geometry>
-    </collision>
-    <visual name='leg_FR_visual'>
-      <origin xyz="0 0 0" rpy="0 0 0"/>
-      <geometry>
-        <box size="${leg_length} ${leg_width} ${leg_height}"/>
-      </geometry>
-    </visual>
-  </link>
-  <link name='leg_FL'>
-    <xacro:box_inertial name="leg_FL" m="${leg_mass}" x="${leg_length}" y="${leg_width}" z="${leg_height}"/>
-    <collision name='leg_FL_collision'>
-      <origin xyz="0 0 0" rpy="0 0 0"/>
-      <geometry>
-        <box size="${leg_length} ${leg_width} ${leg_height}"/>
-      </geometry>
-    </collision>
-    <visual name='leg_FL_visual'>
-      <origin xyz="0 0 0" rpy="0 0 0"/>
-      <geometry>
-        <box size="${leg_length} ${leg_width} ${leg_height}"/>
-      </geometry>
-    </visual>
-  </link>
-    <link name='leg_BR'>
-    <xacro:box_inertial name="leg_FR" m="${leg_mass}" x="${leg_length}" y="${leg_width}" z="${leg_height}"/>
-    <collision name='leg_BR_collision'>
-      <origin xyz="0 0 0" rpy="0 0 0"/>
-      <geometry>
-        <box size="${leg_length} ${leg_width} ${leg_height}"/>
-      </geometry>
-    </collision>
-    <visual name='leg_BR_visual'>
-      <origin xyz="0 0 0" rpy="0 0 0"/>
-      <geometry>
-        <box size="${leg_length} ${leg_width} ${leg_height}"/>
-      </geometry>
-    </visual>
-  </link>
-    <link name='leg_BL'>
-    <xacro:box_inertial name="leg_BL" m="${leg_mass}" x="${leg_length}" y="${leg_width}" z="${leg_height}"/>
-    <collision name='leg_FR_collision'>
-      <origin xyz="0 0 0" rpy="0 0 0"/>
-      <geometry>
-        <box size="${leg_length} ${leg_width} ${leg_height}"/>
-      </geometry>
-    </collision>
-    <visual name='leg_BL_visual'>
-      <origin xyz="0 0 0" rpy="0 0 0"/>
-      <geometry>
-        <box size="${leg_length} ${leg_width} ${leg_height}"/>
-      </geometry>
-    </visual>
-  </link>
-  <joint name="leg_FR_joint" type="fixed">
-    <parent link="chassis"/>
-    <child link="leg_FR"/>
-    <origin xyz="${chassis_length/2 - leg_length/2} ${chassis_width/2 - leg_length/2} ${chassis_height/2 - leg_height/2}"/>
-  </joint>
-  <joint name="leg_FL_joint" type="fixed">
-    <parent link="chassis"/>
-    <child link="leg_FL"/>
-    <origin xyz="-${chassis_length/2 - leg_length/2} ${chassis_width/2 - leg_length/2} ${chassis_height/2 - leg_height/2}"/>
-  </joint>
-  <joint name="leg_BR_joint" type="fixed">
-    <parent link="chassis"/>
-    <child link="leg_BR"/>
-    <origin xyz="${chassis_length/2 - leg_length/2} -${chassis_width/2 - leg_length/2} ${chassis_height/2 - leg_height/2}"/>
-  </joint>
-  <joint name="leg_BL_joint" type="fixed">
-    <parent link="chassis"/>
-    <child link="leg_BL"/>
-    <origin xyz="-${chassis_length/2 - leg_length/2} -${chassis_width/2 - leg_length/2} ${chassis_height/2 - leg_height/2}"/>
-  </joint>
-  <link name='wheel_FR'>
-    <xacro:cylinder_inertial name="wheel_FR" m="${wheel_mass}" r="${wheel_radius}" h="${wheel_width}"/>
-    <collision name='wheel_FR_collision'>
-      <origin xyz="0 0 0" rpy="1.5708 0 0"/>
-      <geometry>
-        <cylinder radius="${wheel_radius}" length="${wheel_width}"/>
-      </geometry>
-    </collision>
-    <visual name='wheel_FR_visual'>
-      <origin xyz="0 0 0" rpy="1.5708 0 0"/>
-      <geometry>
-        <cylinder radius="${wheel_radius}" length="${wheel_width}"/>
-      </geometry>
-    </visual>
-  </link>
+    </link>
   <link name='wheel_FL'>
     <xacro:cylinder_inertial name="wheel_FL" m="${wheel_mass}" r="${wheel_radius}" h="${wheel_width}"/>
     <collision name='wheel_FL_collision'>
       <origin xyz="0 0 0" rpy="1.5708 0 0"/>
-      <geometry>
-        <cylinder radius="${wheel_radius}" length="${wheel_width}"/>
-      </geometry>
+       <mesh>
+            <uri>model://tire/meshes/tire.dae</uri>
+        </mesh>
     </collision>
     <visual name='wheel_FL_visual'>
+      <geometry>
+        <mesh>
+            <uri>model://tire/meshes/tire.dae</uri>
+        </mesh>
+        <!-- <cylinder radius="${wheel_radius}" length="${wheel_width}"/> -->
+      </geometry>
       <origin xyz="0 0 0" rpy="1.5708 0 0"/>
-      <geometry>
-        <cylinder radius="${wheel_radius}" length="${wheel_width}"/>
-      </geometry>
     </visual>
   </link>
-  <link name='wheel_RR'>
-    <xacro:cylinder_inertial name="wheel_RR" m="${wheel_mass}" r="${wheel_radius}" h="${wheel_width}"/>
-    <collision name='wheel_RR_collision'>
-      <origin xyz="0 0 0" rpy="1.5708 0 0"/>
-      <geometry>
-        <cylinder radius="${wheel_radius}" length="${wheel_width}"/>
-      </geometry>
-    </collision>
-    <visual name='wheel_RR_visual'>
-      <origin xyz="0 0 0" rpy="1.5708 0 0"/>
-      <geometry>
-        <cylinder radius="${wheel_radius}" length="${wheel_width}"/>
-      </geometry>
-    </visual>
-  </link>
-  <link name='wheel_RL'>
-    <xacro:cylinder_inertial name="wheel_RL" m="${wheel_mass}" r="${wheel_radius}" h="${wheel_width}"/>
-    <collision name='wheel_RL_collision'>
-      <origin xyz="0 0 0" rpy="1.5708 0 0"/>
-      <geometry>
-        <cylinder radius="${wheel_radius}" length="${wheel_width}"/>
-      </geometry>
-    </collision>
-    <visual name='wheel_RL_visual'>
-      <origin xyz="0 0 0" rpy="1.5708 0 0"/>
-      <geometry>
-        <cylinder radius="${wheel_radius}" length="${wheel_width}"/>
-      </geometry>
-    </visual>
-  </link>
-  <link name='camera_link'>
-    <xacro:box_inertial name="camera_link" m="${camera_mass}" x="${camera_width}" y="${camera_length}" z="${camera_height}"/>
-    <collision name='camera_link_collision'>
-      <geometry>
-        <box size="${camera_length} ${camera_width} ${camera_height}"/>
-      </geometry>
-    </collision>
-    <visual name='camera_link_visual'>
-      <origin xyz="0 0 0" rpy=" 0 0 0"/>
-      <geometry>
-        <box size="${camera_length} ${camera_width} ${camera_height}"/>
-      </geometry>
-    </visual>
-  </link>
-  <link name='downward_camera_link'>
-    <xacro:box_inertial name="downward_camera_link" m="${camera_mass}" x="${camera_width}" y="${camera_length}" z="${camera_height}"/>
-    <collision name='downward_camera_link_collision'>
-      <geometry>
-        <box size="${camera_length} ${camera_width} ${camera_height}"/>
-      </geometry>
-    </collision>
-    <visual name='camera_link_visual'>
-      <origin xyz="0 0 0" rpy=" 0 ${3.1415926/2} 0"/>
-      <geometry>
-        <box size="${5*camera_length} ${2*camera_width} ${camera_height}"/>
-      </geometry>
-    </visual>
-  </link>
-  <joint name="wheel_FR_joint" type="continuous">
+  <joint name="wheel_FL_joint" type="continuous">
     <parent link="chassis"/>
-    <child link="wheel_FR"/>
-    <origin xyz="${chassis_length/2-wheel_radius} -${chassis_width/2+wheel_width/2} ${chassis_height - leg_height - wheel_radius*2.1}"
+    <child link="wheel_FL"/>
+    <origin xyz="${chassis_length/2-wheel_radius} ${chassis_width/2+wheel_width/2} ${chassis_height/2 + wheel_radius*2.1}"
             rpy="0 0 0"/>
     <axis xyz="0 1 0"/>
   </joint>
-  <joint name="wheel_FL_joint" type="continuous">
-    <parent link="chassis"/>
-    <child link="wheel_FL"/>
-    <origin xyz="${chassis_length/2-wheel_radius} ${chassis_width/2+wheel_width/2} ${chassis_height - leg_height - wheel_radius*2.1}"
-            rpy="0 0 0"/>
-    <axis xyz="0 1 0"/>
-  </joint>
-  <joint name="wheel_RR_joint" type="continuous">
-    <parent link="chassis"/>
-    <child link="wheel_RR"/>
-    <origin xyz="-${chassis_length/2-wheel_radius} -${chassis_width/2+wheel_width/2} ${chassis_height - leg_height - wheel_radius*2.1}"
-            rpy="0 0 0"/>
-    <axis xyz="0 1 0"/>
-  </joint>
-  <joint name="wheel_RL_joint" type="continuous">
-    <parent link="chassis"/>
-    <child link="wheel_RL"/>
-    <origin xyz="-${chassis_length/2-wheel_radius} ${chassis_width/2+wheel_width/2} ${chassis_height - leg_height - wheel_radius*2.1}"
-            rpy="0 0 0"/>
-    <axis xyz="0 1 0"/>
-  </joint>
-  <joint name="camera_joint" type="fixed">
-    <parent link="chassis"/>
-    <child link="camera_link"/>
-    <origin xyz="${chassis_length/2} 0 ${chassis_height/2+camera_height/2}"/>
-  </joint>
-  <gazebo reference="chassis">
-    <material>Gazebo/Orange</material>
-  </gazebo>
-  <gazebo reference="camera_link">
-    <material>Gazebo/Blue</material>
-    <sensor type="camera" name="camera_link">
-    <update_rate>30.0</update_rate>
-    <camera name="head">
-      <horizontal_fov>1.3962634</horizontal_fov>
-      <image>
-        <width>800</width>
-        <height>800</height>
-        <format>R8G8B8</format>
-      </image>
-      <clip>
-        <near>0.02</near>
-        <far>300</far>
-      </clip>
-      <noise>
-        <type>gaussian</type>
-        <!-- Noise is sampled independently per pixel on each frame.
-              That pixel's noise value is added to each of its color
-              channels, which at that point lie in the range [0,1]. -->
-        <mean>0.0</mean>
-        <stddev>0.007</stddev>
-      </noise>
-    </camera>
-    <plugin name="camera_controller" filename="libgazebo_ros_camera.so">
-      <alwaysOn>true</alwaysOn>
-      <updateRate>0.0</updateRate>
-      <cameraName>robot/camera</cameraName>
-      <imageTopicName>image_raw</imageTopicName>
-      <cameraInfoTopicName>camera_info</cameraInfoTopicName>
-      <frameName>camera_link</frameName>
-      <hackBaseline>0.07</hackBaseline>
-      <distortionK1>0.0</distortionK1>
-      <distortionK2>0.0</distortionK2>
-      <distortionK3>0.0</distortionK3>
-      <distortionT1>0.0</distortionT1>
-      <distortionT2>0.0</distortionT2>
-    </plugin>
-  </sensor>
-  </gazebo>
-  <joint name="downward_camera_joint" type="fixed">
-    <parent link="chassis"/>
-    <child link="downward_camera_link"/>
-    <origin xyz="0 0 ${-3*camera_height}" rpy="0 1.57 0"/>
-  </joint>
-  <gazebo reference="downward_camera_link">
-    <material>Gazebo/Red</material>
-    <sensor type="camera" name="downward_camera_link">
-    <update_rate>30.0</update_rate>
-    <camera name="head">
-      <horizontal_fov>1.3962634</horizontal_fov>
-      <image>
-        <width>800</width>
-        <height>800</height>
-        <format>R8G8B8</format>
-      </image>
-      <clip>
-        <near>0.02</near>
-        <far>300</far>
-      </clip>
-      <noise>
-        <type>gaussian</type>
-        <!-- Noise is sampled independently per pixel on each frame.
-              That pixel's noise value is added to each of its color
-              channels, which at that point lie in the range [0,1]. -->
-        <mean>0.0</mean>
-        <stddev>0.007</stddev>
-      </noise>
-    </camera>
-    <plugin name="camera_controller" filename="libgazebo_ros_camera.so">
-      <alwaysOn>true</alwaysOn>
-      <updateRate>0.0</updateRate>
-      <cameraName>robot/downward_camera</cameraName>
-      <imageTopicName>downward_image_raw</imageTopicName>
-      <cameraInfoTopicName>downward_camera_info</cameraInfoTopicName>
-      <frameName>downward_camera_link</frameName>
-      <hackBaseline>0.07</hackBaseline>
-      <distortionK1>0.0</distortionK1>
-      <distortionK2>0.0</distortionK2>
-      <distortionK3>0.0</distortionK3>
-      <distortionT1>0.0</distortionT1>
-      <distortionT2>0.0</distortionT2>
-    </plugin>
-  </sensor>
-  </gazebo>
-  <gazebo reference="wheel_FL">
-    <material>Gazebo/Yellow</material>
-  </gazebo>
-  <gazebo reference="wheel_FR">
-    <material>Gazebo/Yellow</material>
-  </gazebo>
-  <gazebo reference="wheel_RL">
-    <material>Gazebo/Yellow</material>
-  </gazebo>
-  <gazebo reference="wheel_RR">
-    <material>Gazebo/Yellow</material>
-  </gazebo>
-  <gazebo>
-    <plugin name="skid_steer_drive_controller" filename="libgazebo_ros_skid_steer_drive.so">
-      <updateRate>100.0</updateRate>
-      <robotNamespace>/</robotNamespace>
-      <leftFrontJoint>wheel_FL_joint</leftFrontJoint>
-      <rightFrontJoint>wheel_FR_joint</rightFrontJoint>
-      <leftRearJoint>wheel_RL_joint</leftRearJoint>
-      <rightRearJoint>wheel_RR_joint</rightRearJoint>
-      <wheelSeparation>0.4</wheelSeparation>
-      <wheelDiameter>0.215</wheelDiameter>
-      <robotBaseFrame>base_link</robotBaseFrame>
-      <torque>20</torque>
-      <topicName>cmd_vel</topicName>
-      <broadcastTF>false</broadcastTF>
-    </plugin>
-  </gazebo>
 </robot>

Commit message: added new scanning algorithm, and updated driving model

File: agrobot_ws/src/agrobot/urdf/robot.xacro (robot description, xacro)
@@ -199,4 +199,18 @@
     <visual name='camera_link_visual'>
       <origin xyz="0 0 0" rpy=" 0 ${3.1415926/2} 0"/>
+      <geometry>
+        <box size="${5*camera_length} ${2*camera_width} ${camera_height}"/>
+      </geometry>
+    </visual>
+  </link>
+<link name='back_camera_link'>
+    <xacro:box_inertial name="back_camera_link" m="${camera_mass}" x="${camera_width}" y="${camera_length}" z="${camera_height}"/>
+    <collision name='back_camera_link_collision'>
+      <geometry>
+        <box size="${camera_length} ${camera_width} ${camera_height}"/>
+      </geometry>
+    </collision>
+    <visual name='camera_link_visual'>
+      <origin xyz="0 0 0" rpy="3.1415926 0 0"/>
       <geometry>
         <box size="${5*camera_length} ${2*camera_width} ${camera_height}"/>
@@ -325,4 +339,49 @@
   </sensor>
   </gazebo>
+  <joint name="back_camera_joint" type="fixed">
+    <parent link="chassis"/>
+    <child link="back_camera_link"/>
+    <origin xyz="${-chassis_length/2} 0 ${chassis_height/2+camera_height/2}" rpy="0 .5 3.1415"/>
+  </joint>
+  <gazebo reference="back_camera_link">
+    <material>Gazebo/Red</material>
+    <sensor type="camera" name="back_camera_link">
+    <update_rate>30.0</update_rate>
+    <camera name="head">
+      <horizontal_fov>1.3962634</horizontal_fov>
+      <image>
+        <width>800</width>
+        <height>800</height>
+        <format>R8G8B8</format>
+      </image>
+      <clip>
+        <near>0.02</near>
+        <far>300</far>
+      </clip>
+      <noise>
+        <type>gaussian</type>
+        <!-- Noise is sampled independently per pixel on each frame.
+              That pixel's noise value is added to each of its color
+              channels, which at that point lie in the range [0,1]. -->
+        <mean>0.0</mean>
+        <stddev>0.007</stddev>
+      </noise>
+    </camera>
+    <plugin name="camera_controller" filename="libgazebo_ros_camera.so">
+      <alwaysOn>true</alwaysOn>
+      <updateRate>0.0</updateRate>
+      <cameraName>robot/back_camera</cameraName>
+      <imageTopicName>back_image_raw</imageTopicName>
+      <cameraInfoTopicName>back_camera_info</cameraInfoTopicName>
+      <frameName>back_camera_link</frameName>
+      <hackBaseline>0.07</hackBaseline>
+      <distortionK1>0.0</distortionK1>
+      <distortionK2>0.0</distortionK2>
+      <distortionK3>0.0</distortionK3>
+      <distortionT1>0.0</distortionT1>
+      <distortionT2>0.0</distortionT2>
+    </plugin>
+  </sensor>
+  </gazebo>
   <gazebo reference="wheel_FL">
     <material>Gazebo/Yellow</material>
