Commit message: re-organized folder structure for all algorithms

File: agrobot_ws/src/agrobot/urdf/agrobot.xacro (robot description, xacro)
@@ -3,17 +3,27 @@
   <xacro:property name="chassis_x" value="1"/>
   <xacro:property name="chassis_y" value="0.65"/>
-  <xacro:property name="chassis_z" value="0.1"/>
+  <xacro:property name="chassis_z" value="0.06"/>
   <xacro:property name="chassis_mass" value="50"/>
   <xacro:property name="wheel_radius" value="0.1"/>
   <xacro:property name="wheel_width" value="0.05"/>
   <xacro:property name="wheel_mass" value="5"/>
-  <xacro:property name="leg_x" value="0.1"/>
-  <xacro:property name="leg_y" value="0.1"/>
+  <xacro:property name="leg_x" value="0.06"/>
+  <xacro:property name="leg_y" value="0.06"/>
   <xacro:property name="leg_z" value="0.75"/>
   <xacro:property name="leg_mass" value="10"/>
+  <xacro:property name="camera_x" value="0.05"/>
+  <xacro:property name="camera_y" value="0.08"/>
+  <xacro:property name="camera_z" value="0.03"/>
+  <xacro:property name="camera_mass" value="0.1"/>
   <xacro:property name="steerer_size" value="0.1"/>
   <xacro:property name="steerer_mass" value="2"/>
+  <xacro:property name="pi" value="3.1415926"/>
   <xacro:include filename="$(find agrobot)/urdf/macros.xacro"/>
   <xacro:include filename="$(find agrobot)/urdf/materials.xacro"/>
+  <gazebo>
+    <plugin name="gazebo_ros_control" filename="libgazebo_ros_control.so">
+        <robotNamespace>/agrobot</robotNamespace>
+    </plugin>
+  </gazebo>
   <link name='chassis'>
     <collision name='chassis_collision'>
@@ -29,4 +39,8 @@
     </visual>
   </link>
+  <gazebo reference="chassis">
+    <material>Gazebo/Yellow</material>
+  </gazebo>
+<!--
   <link name='stand'>
     <xacro:box_inertial name="stand" m="${100}" x="${leg_x}" y="${leg_y}" z="${leg_z}"/>
@@ -49,4 +63,5 @@
     <origin xyz="${0} ${0} ${-chassis_z/2 - leg_z*1.5/2}"/>
   </joint>
+ -->
   <link name='leg_FL'>
     <xacro:box_inertial name="leg_FL" m="${leg_mass}" x="${leg_x}" y="${leg_y}" z="${leg_z}"/>
@@ -64,4 +79,7 @@
     </visual>
   </link>
+  <gazebo reference="leg_FL">
+    <material>Gazebo/Red</material>
+  </gazebo>
   <joint name="leg_FL_joint" type="fixed">
     <parent link="chassis"/>
@@ -84,4 +102,7 @@
     </visual>
   </link>
+  <gazebo reference="steerer_FL">
+    <material>Gazebo/Red</material>
+  </gazebo>
   <joint name="wheel_FL_position_joint" type="continuous">
     <parent link="leg_FL"/>
@@ -90,4 +111,14 @@
     <axis xyz="0 0 1"/>
   </joint>
+  <transmission name="wheel_FL_steerer_transmission">
+    <type>transmission_interface/SimpleTransmission</type>
+    <joint name="wheel_FL_position_joint">
+        <hardwareInterface>hardware_interface/EffortJointInterface</hardwareInterface>
+    </joint>
+    <actuator name="FL_position_motor">
+        <hardwareInterface>hardware_interface/EffortJointInterface</hardwareInterface>
+        <mechanicalReduction>1</mechanicalReduction>
+    </actuator>
+  </transmission>
   <link name='wheel_FL'>
     <xacro:cylinder_inertial name="wheel_FL" m="${wheel_mass}" r="${wheel_radius}" h="${wheel_width}"/>
@@ -103,8 +134,10 @@
       <geometry>
         <mesh filename="package://agrobot/models/tire/meshes/tire.dae" scale="0.5 0.5 0.5"/>
-        <!-- <cylinder radius="${wheel_radius}" length="${wheel_width}"/> -->
-      </geometry>
-    </visual>
-  </link>
+      </geometry>
+    </visual>
+  </link>
+  <gazebo reference="wheel_FL">
+    <material>Gazebo/Black</material>
+  </gazebo>
   <joint name="wheel_FL_velocity_joint" type="continuous">
     <parent link="steerer_FL"/>
@@ -114,53 +147,417 @@
     <axis xyz="0 1 0"/>
   </joint>
-  <gazebo reference="chassis">
+  <transmission name="wheel_FL_velocity_transmission">
+    <type>transmission_interface/SimpleTransmission</type>
+    <joint name="wheel_FL_velocity_joint">
+        <hardwareInterface>hardware_interface/EffortJointInterface</hardwareInterface>
+    </joint>
+    <actuator name="FL_velocity_motor">
+        <hardwareInterface>hardware_interface/EffortJointInterface</hardwareInterface>
+        <mechanicalReduction>1</mechanicalReduction>
+    </actuator>
+  </transmission>
+  <!-- ##################### all components for FR leg ###############################-->
+  <link name='leg_FR'>
+    <xacro:box_inertial name="leg_FR" m="${leg_mass}" x="${leg_x}" y="${leg_y}" z="${leg_z}"/>
+    <collision name='leg_FR_collision'>
+      <origin xyz="0 0 0" rpy="0 0 0"/>
+      <geometry>
+        <box size="${leg_x} ${leg_y} ${leg_z}"/>
+      </geometry>
+    </collision>
+    <visual name='leg_FR_visual'>
+      <origin xyz="0 0 ${wheel_radius*1.1/2}" rpy="0 0 0"/>
+      <geometry>
+        <box size="${leg_x} ${leg_y} ${leg_z-wheel_radius*1.1}"/>
+      </geometry>
+    </visual>
+  </link>
+  <gazebo reference="leg_FR">
+    <material>Gazebo/Red</material>
+  </gazebo>
+  <joint name="leg_FR_joint" type="fixed">
+    <parent link="chassis"/>
+    <child link="leg_FR"/>
+    <origin xyz="${chassis_x/2 - leg_x/2} ${-chassis_y/2 + leg_y/2} ${-chassis_z/2 - leg_z/2}"/>
+  </joint>
+  <link name='steerer_FR'>
+    <xacro:box_inertial name="steerer_FR" m="${steerer_mass}" x="${steerer_size}" y="${steerer_size}" z="${steerer_size}"/>
+    <collision name='steerer_FR_collision'>
+      <origin xyz="0 0 0" rpy="0 0 0"/>
+      <geometry>
+        <box size="${steerer_size} ${steerer_size} ${steerer_size}"/>
+      </geometry>
+    </collision>
+    <visual name='steerer_FR_visual'>
+      <origin xyz="0 0 0" rpy="0 0 0"/>
+      <geometry>
+        <box size="${steerer_size/5} ${steerer_size/5} ${steerer_size/5}"/>
+      </geometry>
+    </visual>
+  </link>
+  <gazebo reference="steerer_FR">
+    <material>Gazebo/Red</material>
+  </gazebo>
+  <joint name="wheel_FR_position_joint" type="continuous">
+    <parent link="leg_FR"/>
+    <child link="steerer_FR"/>
+    <origin xyz="${0} ${0} ${-leg_z/2 - leg_x/2}"/>
+    <axis xyz="0 0 1"/>
+  </joint>
+  <transmission name="wheel_FR_steerer_transmission">
+    <type>transmission_interface/SimpleTransmission</type>
+    <joint name="wheel_FR_position_joint">
+        <hardwareInterface>hardware_interface/EffortJointInterface</hardwareInterface>
+    </joint>
+    <actuator name="FR_position_motor">
+        <hardwareInterface>hardware_interface/EffortJointInterface</hardwareInterface>
+        <mechanicalReduction>1</mechanicalReduction>
+    </actuator>
+  </transmission>
+  <link name='wheel_FR'>
+    <xacro:cylinder_inertial name="wheel_FR" m="${wheel_mass}" r="${wheel_radius}" h="${wheel_width}"/>
+    <dynamics damping="0.01" friction="1.0"/>
+    <collision name='wheel_FR_collision'>
+      <origin xyz="0 0 0" rpy="1.5708 0 0"/>
+      <geometry>
+        <cylinder radius="${wheel_radius}" length="${wheel_width}"/>
+      </geometry>
+    </collision>
+    <visual name='wheel_FR_visual'>
+      <origin xyz="0 0 0" rpy="0 0 0"/>
+      <geometry>
+        <mesh filename="package://agrobot/models/tire/meshes/tire.dae" scale="0.5 0.5 0.5"/>
+      </geometry>
+    </visual>
+  </link>
+  <gazebo reference="wheel_FR">
+    <material>Gazebo/Black</material>
+  </gazebo>
+  <joint name="wheel_FR_velocity_joint" type="continuous">
+    <parent link="steerer_FR"/>
+    <child link="wheel_FR"/>
+    <origin xyz="0 0 0"
+            rpy="0 0 0"/>
+    <axis xyz="0 1 0"/>
+  </joint>
+  <transmission name="wheel_FR_velocity_transmission">
+    <type>transmission_interface/SimpleTransmission</type>
+    <joint name="wheel_FR_velocity_joint">
+        <hardwareInterface>hardware_interface/EffortJointInterface</hardwareInterface>
+    </joint>
+    <actuator name="FR_velocity_motor">
+        <hardwareInterface>hardware_interface/EffortJointInterface</hardwareInterface>
+        <mechanicalReduction>1</mechanicalReduction>
+    </actuator>
+  </transmission>
+  <!-- ################# BL Leg ############################# -->
+  <link name='leg_BL'>
+    <xacro:box_inertial name="leg_BL" m="${leg_mass}" x="${leg_x}" y="${leg_y}" z="${leg_z}"/>
+    <collision name='leg_BL_collision'>
+      <origin xyz="0 0 0" rpy="0 0 0"/>
+      <geometry>
+        <box size="${leg_x} ${leg_y} ${leg_z}"/>
+      </geometry>
+    </collision>
+    <visual name='leg_BL_visual'>
+      <origin xyz="0 0 ${wheel_radius*1.1/2}" rpy="0 0 0"/>
+      <geometry>
+        <box size="${leg_x} ${leg_y} ${leg_z-wheel_radius*1.1}"/>
+      </geometry>
+    </visual>
+  </link>
+  <gazebo reference="leg_BL">
+    <material>Gazebo/Red</material>
+  </gazebo>
+  <joint name="leg_BL_joint" type="fixed">
+    <parent link="chassis"/>
+    <child link="leg_BL"/>
+    <origin xyz="${-chassis_x/2 + leg_x/2} ${chassis_y/2 - leg_y/2} ${-chassis_z/2 - leg_z/2}"/>
+  </joint>
+  <link name='steerer_BL'>
+    <xacro:box_inertial name="steerer_BL" m="${steerer_mass}" x="${steerer_size}" y="${steerer_size}" z="${steerer_size}"/>
+    <collision name='steerer_BL_collision'>
+      <origin xyz="0 0 0" rpy="0 0 0"/>
+      <geometry>
+        <box size="${steerer_size} ${steerer_size} ${steerer_size}"/>
+      </geometry>
+    </collision>
+    <visual name='steerer_BL_visual'>
+      <origin xyz="0 0 0" rpy="0 0 0"/>
+      <geometry>
+        <box size="${steerer_size/5} ${steerer_size/5} ${steerer_size/5}"/>
+      </geometry>
+    </visual>
+  </link>
+  <gazebo reference="steerer_BL">
+    <material>Gazebo/Red</material>
+  </gazebo>
+  <joint name="wheel_BL_position_joint" type="continuous">
+    <parent link="leg_BL"/>
+    <child link="steerer_BL"/>
+    <origin xyz="${0} ${0} ${-leg_z/2 - leg_x/2}"/>
+    <axis xyz="0 0 1"/>
+  </joint>
+  <transmission name="wheel_BL_steerer_transmission">
+    <type>transmission_interface/SimpleTransmission</type>
+    <joint name="wheel_BL_position_joint">
+        <hardwareInterface>hardware_interface/EffortJointInterface</hardwareInterface>
+    </joint>
+    <actuator name="BL_position_motor">
+        <hardwareInterface>hardware_interface/EffortJointInterface</hardwareInterface>
+        <mechanicalReduction>1</mechanicalReduction>
+    </actuator>
+  </transmission>
+  <link name='wheel_BL'>
+    <xacro:cylinder_inertial name="wheel_BL" m="${wheel_mass}" r="${wheel_radius}" h="${wheel_width}"/>
+    <dynamics damping="0.01" friction="1.0"/>
+    <collision name='wheel_BL_collision'>
+      <origin xyz="0 0 0" rpy="1.5708 0 0"/>
+      <geometry>
+        <cylinder radius="${wheel_radius}" length="${wheel_width}"/>
+      </geometry>
+    </collision>
+    <visual name='wheel_BL_visual'>
+      <origin xyz="0 0 0" rpy="0 0 0"/>
+      <geometry>
+        <mesh filename="package://agrobot/models/tire/meshes/tire.dae" scale="0.5 0.5 0.5"/>
+      </geometry>
+    </visual>
+  </link>
+  <gazebo reference="wheel_BL">
+    <material>Gazebo/Black</material>
+  </gazebo>
+  <joint name="wheel_BL_velocity_joint" type="continuous">
+    <parent link="steerer_BL"/>
+    <child link="wheel_BL"/>
+    <origin xyz="0 0 0"
+            rpy="0 0 0"/>
+    <axis xyz="0 1 0"/>
+  </joint>
+  <transmission name="wheel_BL_velocity_transmission">
+    <type>transmission_interface/SimpleTransmission</type>
+    <joint name="wheel_BL_velocity_joint">
+        <hardwareInterface>hardware_interface/EffortJointInterface</hardwareInterface>
+    </joint>
+    <actuator name="BL_velocity_motor">
+        <hardwareInterface>hardware_interface/EffortJointInterface</hardwareInterface>
+        <mechanicalReduction>1</mechanicalReduction>
+    </actuator>
+  </transmission>
+  <!-- ################# BR Leg ############################# -->
+  <link name='leg_BR'>
+    <xacro:box_inertial name="leg_BR" m="${leg_mass}" x="${leg_x}" y="${leg_y}" z="${leg_z}"/>
+    <collision name='leg_BR_collision'>
+      <origin xyz="0 0 0" rpy="0 0 0"/>
+      <geometry>
+        <box size="${leg_x} ${leg_y} ${leg_z}"/>
+      </geometry>
+    </collision>
+    <visual name='leg_BR_visual'>
+      <origin xyz="0 0 ${wheel_radius*1.1/2}" rpy="0 0 0"/>
+      <geometry>
+        <box size="${leg_x} ${leg_y} ${leg_z-wheel_radius*1.1}"/>
+      </geometry>
+    </visual>
+  </link>
+  <gazebo reference="leg_BR">
+    <material>Gazebo/Red</material>
+  </gazebo>
+  <joint name="leg_BR_joint" type="fixed">
+    <parent link="chassis"/>
+    <child link="leg_BR"/>
+    <origin xyz="${-chassis_x/2 + leg_x/2} ${-chassis_y/2 + leg_y/2} ${-chassis_z/2 - leg_z/2}"/>
+  </joint>
+  <link name='steerer_BR'>
+    <xacro:box_inertial name="steerer_BR" m="${steerer_mass}" x="${steerer_size}" y="${steerer_size}" z="${steerer_size}"/>
+    <collision name='steerer_BR_collision'>
+      <origin xyz="0 0 0" rpy="0 0 0"/>
+      <geometry>
+        <box size="${steerer_size} ${steerer_size} ${steerer_size}"/>
+      </geometry>
+    </collision>
+    <visual name='steerer_BR_visual'>
+      <origin xyz="0 0 0" rpy="0 0 0"/>
+      <geometry>
+        <box size="${steerer_size/5} ${steerer_size/5} ${steerer_size/5}"/>
+      </geometry>
+    </visual>
+  </link>
+  <gazebo reference="steerer_BR">
+    <material>Gazebo/Red</material>
+  </gazebo>
+  <joint name="wheel_BR_position_joint" type="continuous">
+    <parent link="leg_BR"/>
+    <child link="steerer_BR"/>
+    <origin xyz="${0} ${0} ${-leg_z/2 - leg_x/2}"/>
+    <axis xyz="0 0 1"/>
+  </joint>
+  <transmission name="wheel_BR_steerer_transmission">
+    <type>transmission_interface/SimpleTransmission</type>
+    <joint name="wheel_BR_position_joint">
+        <hardwareInterface>hardware_interface/EffortJointInterface</hardwareInterface>
+    </joint>
+    <actuator name="BR_position_motor">
+        <hardwareInterface>hardware_interface/EffortJointInterface</hardwareInterface>
+        <mechanicalReduction>1</mechanicalReduction>
+    </actuator>
+  </transmission>
+  <link name='wheel_BR'>
+    <xacro:cylinder_inertial name="wheel_BR" m="${wheel_mass}" r="${wheel_radius}" h="${wheel_width}"/>
+    <dynamics damping="0.01" friction="1.0"/>
+    <collision name='wheel_BR_collision'>
+      <origin xyz="0 0 0" rpy="1.5708 0 0"/>
+      <geometry>
+        <cylinder radius="${wheel_radius}" length="${wheel_width}"/>
+      </geometry>
+    </collision>
+    <visual name='wheel_BR_visual'>
+      <origin xyz="0 0 0" rpy="0 0 0"/>
+      <geometry>
+        <mesh filename="package://agrobot/models/tire/meshes/tire.dae" scale="0.5 0.5 0.5"/>
+      </geometry>
+    </visual>
+  </link>
+  <gazebo reference="wheel_BR">
+    <material>Gazebo/Black</material>
+  </gazebo>
+  <joint name="wheel_BR_velocity_joint" type="continuous">
+    <parent link="steerer_BR"/>
+    <child link="wheel_BR"/>
+    <origin xyz="0 0 0"
+            rpy="0 0 0"/>
+    <axis xyz="0 1 0"/>
+  </joint>
+  <transmission name="wheel_BR_velocity_transmission">
+    <type>transmission_interface/SimpleTransmission</type>
+    <joint name="wheel_BR_velocity_joint">
+        <hardwareInterface>hardware_interface/EffortJointInterface</hardwareInterface>
+    </joint>
+    <actuator name="BR_velocity_motor">
+        <hardwareInterface>hardware_interface/EffortJointInterface</hardwareInterface>
+        <mechanicalReduction>1</mechanicalReduction>
+    </actuator>
+  </transmission>
+<!-- ###########################################################################################
+                                Cameras and Sensors
+############################################################################################ -->
+ <link name='front_camera'>
+    <xacro:box_inertial name="front_camera" m="${camera_mass}" x="${camera_x}" y="${camera_y}" z="${camera_z}"/>
+    <collision name='front_camera_collision'>
+      <geometry>
+        <box size="${camera_x} ${camera_y} ${camera_z}"/>
+      </geometry>
+    </collision>
+    <visual name='front_camera_visual'>
+      <origin xyz="0 0 0" rpy="0 0 0"/>
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
Commit message: added left and right cameras

File: agrobot_ws/src/agrobot/urdf/agrobot.xacro (robot description, xacro)
@@ -442,4 +442,5 @@
                                 Cameras and Sensors
 ############################################################################################ -->
+<!-- **************************** front camera ********************************************* -->
  <link name='front_camera'>
     <xacro:box_inertial name="front_camera" m="${camera_mass}" x="${camera_x}" y="${camera_y}" z="${camera_z}"/>
@@ -501,4 +502,5 @@
   </sensor>
   </gazebo>
+<!-- **************************** downward camera ********************************************* -->
    <link name='downward_camera'>
     <xacro:box_inertial name="downward_camera" m="${camera_mass}" x="${camera_x}" y="${camera_y}" z="${camera_z}"/>
@@ -561,3 +563,159 @@
   </sensor>
   </gazebo>
+<!-- **************************** left side camera ********************************************* -->
+   <link name='left_side_camera'>
+    <xacro:box_inertial name="left_side_camera" m="${camera_mass}" x="${camera_x}" y="${camera_y}" z="${camera_z}"/>
+    <collision name='left_side_camera_collision'>
+      <geometry>
+        <box size="${camera_x} ${camera_y} ${camera_z}"/>
+      </geometry>
+    </collision>
+    <visual name='left_side_camera_visual'>
+      <origin xyz="0 0 0" rpy="0 0 0"/>
+      <geometry>
+        <box size="${camera_x} ${camera_y} ${camera_z}"/>
+      </geometry>
+    </visual>
+  </link>
+  <joint name="left_side_camera_joint" type="fixed">
+    <parent link="leg_BL"/>
+    <child link="left_side_camera"/>
+    <origin xyz="0 ${leg_y/2} -${leg_z*1/3}" rpy="0 0 ${pi/2}"/>
+  </joint>
+  <gazebo reference="left_side_camera">
+    <material>Gazebo/Blue</material>
+    <sensor type="camera" name="camera_link">
+    <update_rate>30.0</update_rate>
+    <camera name="left_side_camera">
+      <horizontal_fov>1.3962634</horizontal_fov>
+      <image>
+        <width>400</width>
+        <height>400</height>
+        <format>R8G8B8</format>
+      </image>
+      <clip>
+        <near>0.02</near>
+        <far>300</far>
+      </clip>
+      <noise>
+        <type>gaussian</type>
+        <!-- Noise is sampled independently per pixel on each frame.
+              That pixel's noise value is added to each of its color
+              channels, which at that point lie in the range [0,1]. -->
+        <mean>0.0</mean>
+        <stddev>0.007</stddev>
+      </noise>
+    </camera>
+    <plugin name="camera_controller" filename="libgazebo_ros_camera.so">
+      <alwaysOn>true</alwaysOn>
+      <updateRate>0.0</updateRate>
+      <cameraName>agrobot/left_side_camera</cameraName>
+      <imageTopicName>image</imageTopicName>
+      <cameraInfoTopicName>left_side_camera_info</cameraInfoTopicName>
+      <frameName>left_side_camera_frame</frameName>
+      <hackBaseline>0.07</hackBaseline>
+      <distortionK1>0.0</distortionK1>
+      <distortionK2>0.0</distortionK2>
+      <distortionK3>0.0</distortionK3>
+      <distortionT1>0.0</distortionT1>
+      <distortionT2>0.0</distortionT2>
+    </plugin>
+  </sensor>
+  </gazebo>
+<!-- **************************** right side camera ********************************************* -->
+<link name='right_side_camera'>
+    <xacro:box_inertial name="right_side_camera" m="${camera_mass}" x="${camera_x}" y="${camera_y}" z="${camera_z}"/>
+    <collision name='right_side_camera_collision'>
+      <geometry>
+        <box size="${camera_x} ${camera_y} ${camera_z}"/>
+      </geometry>
+    </collision>
+    <visual name='right_side_camera_visual'>
+      <origin xyz="0 0 0" rpy="0 0 0"/>
+      <geometry>
+        <box size="${camera_x} ${camera_y} ${camera_z}"/>
+      </geometry>
+    </visual>
+  </link>
+  <joint name="right_side_camera_joint" type="fixed">
+    <parent link="leg_BR"/>
+    <child link="right_side_camera"/>
+    <origin xyz="0 -${leg_y/2} -${leg_z*1/3}" rpy="0 0 -${pi/2}"/>
+  </joint>
+  <gazebo reference="right_side_camera">
+    <material>Gazebo/Blue</material>
+    <sensor type="camera" name="camera_link">
+    <update_rate>30.0</update_rate>
+    <camera name="right_side_camera">
+      <horizontal_fov>1.3962634</horizontal_fov>
+      <image>
+        <width>400</width>
+        <height>400</height>
+        <format>R8G8B8</format>
+      </image>
+      <clip>
+        <near>0.02</near>
+        <far>300</far>
+      </clip>
+      <noise>
+        <type>gaussian</type>
+        <!-- Noise is sampled independently per pixel on each frame.
+              That pixel's noise value is added to each of its color
+              channels, which at that point lie in the range [0,1]. -->
+        <mean>0.0</mean>
+        <stddev>0.007</stddev>
+      </noise>
+    </camera>
+    <plugin name="camera_controller" filename="libgazebo_ros_camera.so">
+      <alwaysOn>true</alwaysOn>
+      <updateRate>0.0</updateRate>
+      <cameraName>agrobot/right_side_camera</cameraName>
+      <imageTopicName>image</imageTopicName>
+      <cameraInfoTopicName>right_side_camera_info</cameraInfoTopicName>
+      <frameName>right_side_camera_frame</frameName>
+      <hackBaseline>0.07</hackBaseline>
+      <distortionK1>0.0</distortionK1>
+      <distortionK2>0.0</distortionK2>
+      <distortionK3>0.0</distortionK3>
+      <distortionT1>0.0</distortionT1>
+      <distortionT2>0.0</distortionT2>
+    </plugin>
+  </sensor>
+  </gazebo>
+<!-- **************************** imu sensor ********************************************* -->
+<joint name="imu_joint" type="fixed">
+    <axis xyz="1 0 0"/> <!-- 0 1 0 -->
+    <origin xyz="0 0 ${chassis_z}"/>
+    <parent link="chassis"/>
+    <child link="imu_link"/>
+  </joint>
+<link name="imu_link">
+  <inertial>
+    <mass value="0.001"/>
+    <origin rpy="0 0 0" xyz="0 0 0"/>
+    <inertia ixx="0.0001" ixy="0" ixz="0" iyy="0.000001" iyz="0" izz="0.0001"/>
+  </inertial>
+  <visual>
+    <origin rpy="0 0 0" xyz="0 0 0"/>
+    <geometry>
+      <box size="0.001 0.001 0.001"/>
+    </geometry>
+  </visual>
+  <collision>
+    <origin rpy="0 0 0" xyz="0 0 0"/>
+    <geometry>
+      <box size=".1 .1 .1"/>
+    </geometry>
+  </collision>
+</link>
+  <gazebo>
+    <plugin name="imu_plugin" filename="libgazebo_ros_imu.so">
+      <alwaysOn>true</alwaysOn>
+      <bodyName>imu_link</bodyName>
+      <topicName>agrobot/imu</topicName>
+      <serviceName>imu_service</serviceName>
+      <gaussianNoise>0.0</gaussianNoise>
+      <updateRate>20.0</updateRate>
+    </plugin>
+  </gazebo>
 </robot>
